File: UpBoard/X/R1/UpBoardXR1.sch (EAGLE design)
At the start: 59 parts, among them CN1 100nF, CN2 100nF, CN3 100nF, CN4 100nF, IC1 SAM3X8E(ARDUINO), J1 2POSTERMINALBLOCK.25"PITCH, Q6 2N7002E, X1 16POS_RIBBON, X2 16POS_RIBBON, X3 16POS_RIBBON, X4 16POS_RIBBON, Y1 FH1200001, Y2 ABS05

Commit message: Update R1
Parts:
- added RST_EN1: 1K, resistor:R-US_R0402
- US1: device adafruit:USBMINIB -> SparkFun-Connectors:USB_MICRO-B_FEMALE-SMT
Connections:
- removed net N$13: U$4.CS
- removed net N$14: U$4.WP
- removed net N$15: U$4.HOLD
- net 3.3V: now also RST_EN1.1, XA1.P$2
- net D6: now also U$4.HOLD
- net D7: now also RST_EN1.2, U$4.CS
- net D8: now also U$4.WP
- net HV: no longer XA1.P$2, XA1.P$3
- net MISO: no longer U$4.DI
- net MOSI: now also U$4.DI
- net N$3: no longer U$4.CLK
- net SCK: now also U$4.CLK
Other:
- moved on the sheet: X1, X2, X3, X4

Commit message: Connected Flash corrctly, changed sheet size
Parts:
- removed R37: 0R, resistor:R-US_R0402
- removed RST_EN1: 1K, resistor:R-US_R0402
- removed US1: (no value), SparkFun-Connectors:USB_MICRO-B_FEMALE-SMT
- added J2: (no value), SparkFun-Connectors:CONN_02
- added RN4: 1K, resistor-net:CTS742C083
- added U$5: MICROUSB_5POS_SMT, CPSS_CONNECTOR:MICROUSB_5POS_SMT
- R38: value 0R -> 220R
Connections:
- net 3.3V: now also RN4.7, RN4.8; no longer RST_EN1.1
- net D+: now also U$5.D+; no longer US1.D+
- net D-: now also U$5.D-; no longer US1.D-
- net D6: now also RN4.1
- net D7: now also J2.1, RN4.2; no longer RST_EN1.2
- net D8: now also J2.2, RN4.4
- net GND: now also RN4.5, U$5.GND; no longer R37.2, US1.GND
- net TST: no longer R37.1
- net UOTGID: now also U$5.ID; no longer US1.ID
- net VBUS: now also U$5.VCC; no longer US1.VBUS
Other:
- note added: "B"
- note removed: "C"
- moved on the sheet: C1, C12, C13, C14, C15, C16, C4, C5, C6, C7, C8, CN1G$2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

Commit message: Finished routing traces, front silkscreen.
Parts:
- removed C13, C14: 10uF, resistor:CPOL-EUA/3216-18R
- removed ERASE_EN, RST_EN: 0R, resistor:R-US_R0402
- removed LED4: (no value), led:LEDCHIPLED_0805
- removed Q6: 2N7002E, UpBoard B:2N7002E
- removed R17: 10k, resistor:R-US_R0603
- removed R38: 220R, resistor:R-US_R0402
- removed U$1, U$3: BC857BV-7, CPSS_IC:BC857BV-7
- added C2, C3: 22pF, resistor:C-EUC0603
- added C9: 10uF, resistor:CPOL-EUA/3216-18R
- added Q1, Q2: MBT3904DW2T1, CPSS_IC:MBT3904DW2T1
- added R1, R2: 39, resistor:R-US_R0603
- added U$6, U$7: SOLBRDG, CPSS_CONNECTOR:SOLBRDG
- C6: value 22pF -> 10n
- C7: value 22pF -> 100n
- C8: value 10n -> 10uF; device resistor:C-EUC0603 -> resistor:CPOL-EUA/3216-18R
- R3, R4: value 39 -> 220R; device resistor:R-US_R0603 -> resistor:R-US_R0402
- RN1: value 10K -> 65R
- RN2: value 1k -> 4.7K
- RN3: value 10K -> 100K
- RN4: value 1K -> 100K
- renumbered C15 to C10, C16 to C11, J1 to XP1, LSP1 to GND, R15 to R5, R39 to R6, U$4 to IC2, U$5 to XU1
Connections:
- net N$17 renamed D26
- removed net N$38: LED1.C, U$3G$1.C
- removed net N$8: LED3.C, U$1G$1.C
- removed net VIN: U$3G$1.+
- new net N$1: LED3.C, RN1.2
- new net N$11: Q1G$2.C, RN1.6
- new net N$12: Q1G$1.C, RN1.5
- new net N$5: PWR.C, RN1.1
- net 1.8V: now also C12.+, CN1G$1.1, CN1G$2.1, CN3G$3.1, CN3G$4.1; no longer C13.+, CN2G$1.1, CN2G$2.1, CN2G$3.1, CN2G$4.1
- net 3.3V: now also C6.1, C7.2, C8.+, CN1G$3.1, CN1G$4.1, R4.2, RN4.5, RN4.6, U$6.P$2; no longer C12.+, C8.1, CN3G$3.1, CN3G$4.1, ERASE_EN.2, LED4.A, RN1.5, RN1.6, RN1.7, RN1.8
- net 5V: now also C3.1, C4.1, C9.1, IC1.OUT; no longer C7.1, U$2.OUT
- net BATT_5V: now also C8.1, IC1.IN1; no longer U$1G$1.VOUT, U$2.IN1
- net D+: now also R1.1; no longer R3.1
- net D-: now also R2.1; no longer R4.1
- net D10: now also U$2.2-CD/DAT3; no longer RN3.1, U$1G$2.B
- net D11: now also Q1G$1.B; no longer U$1G$1.B, U$2.2-CD/DAT3
- net D12: now also Q1G$2.B; no longer U$3G$2.B
- net D13: now also Q2G$1.B; no longer U$3G$1.B
- net D6: no longer RN4.1
- net D7: now also R4.1; no longer RN4.2
- net D8: no longer RN4.4
- net D9: now also Q2G$2.B, RN3.1; no longer Q6.G, R17.1
- net GND: now also C2.2, C3.2, C7.1, C8.-, C8.2, C9.-, C9.2, CN1G$1.2, CN1G$2.2, CN1G$3.2, CN1G$4.2, CN2G$2.1, CN2G$3.1, CN2G$4.1, IC1.D1, Q1G$1.E, Q1G$2.E, Q2G$1.E, Q2G$2.E, R1.2, R3.2, RN1.8, U$7.P$2; no longer C13.-, C14.-, CN1G$2.1, CN1G$3.1, CN1G$4.1, CN2G$1.2, CN2G$2.2, CN2G$3.2, CN2G$4.2, PWR.C, Q6.S, R17.2, R38.2, RN4.5, RST_EN.2, U$1G$1.E, U$1G$1.GND, U$1G$2.E, U$2.D1, U$2.GND, U$3G$1.E, U$3G$2.E
- net HV: now also C7.1; no longer C1.1, U$3G$1.-
- net JTAG_SEL: now also R3.1; no longer R38.1
- net JTAG_TCK: now also RN4.2; no longer RN1.2
- net JTAG_TDI: now also RN4.3; no longer RN1.3
- net JTAG_TMS: now also RN4.1; no longer RN1.1
- net M_RESET: now also C6.2, RN4.4; no longer C8.2, RN1.4
- net N$10: now also Q2G$1.C, RN1.7; no longer LED4.C, U$1G$2.C
- net N$2: now also C5.1, R1.2; no longer R3.2, U$1G$1.VIN
- net N$22: now also U$6.P$1; no longer ERASE_EN.1
- net N$3: now also IC1.ILIM, LED2.C, R1.1, RN1.3; no longer U$2.ILIM
- net N$33: now also Q2G$2.C; no longer Q6.D
- net N$35: now also C2.1; no longer C7.1
- net N$36: now also C3.1; no longer C6.1
- net N$6: now also U$7.P$1; no longer RST_EN.1
- net N$7: now also LED1.C, RN1.4; no longer LED2.C, U$3G$2.C
- net N$9: now also R2.2; no longer R4.2
- net USB_FILTERED: now also C2.1, IC1.IN2; no longer C5.1, U$2.IN2
- net VBUS: now also C1.1; no longer C4.1
- net VDDANA: now also CN2G$3.2; no longer CN1G$3.2
- net VDDPLL: now also CN2G$2.2; no longer CN1G$2.2
- net VDDUTMI: now also C9.+, CN2G$4.2; no longer C14.+, CN1G$4.2
Other:
- note removed: "File: UpBoardX.sch"
- moved on the sheet: C12, C6, C7, CN1G$2, CN1G$3, CN1G$4, CN2G$2, CN2G$3, CN2G$4, CN3G$1, CN3G$2, CN3G$3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

Commit message: Fixed refdes
Parts:
- removed D7: (no value), zetex:DSOD323
- added D1: (no value), zetex:DSOD323
- renumbered D8 to D2, J2 to JP3, U$2 to SD1, U$6 to SJ3, U$7 to SJ2
Connections:
- new net VIN: D1.+
- net HV: now also D1.-, D1.A; no longer D7.A
- net LS_DRIVE: now also D1.C; no longer D7.C
Changed lines of the file:
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@@
 <drawing>
 <settings>
-<setting alwaysvectorfont="no"/>
+<setting alwaysvectorfont="yes"/>
 <setting keepoldvectorfont="yes"/>
 <setting verticaltext="up"/>
@@
 <parts>
 <part name="IC1" library="ATSAM3X" deviceset="SAM3X8E(ARDUINO)" device=""/>
-<part name="U$2" library="UpBoard B" deviceset="CONN_MICROSD" device=""/>
+<part name="SD1" library="UpBoard B" deviceset="CONN_MICROSD" device=""/>
 <part name="XP1" library="terminal_block" deviceset="2POSTERMINALBLOCK" device=".25&quot;PITCH"/>
 <part name="R1" library="resistor" deviceset="R-US_" device="R0603" value="39"/>
@@
 <part name="C1" library="resistor" deviceset="C-EU" device="C0603" value="10pF"/>
 <part name="R5" library="resistor" deviceset="R-US_" device="R0603" value="6.8K"/>
-<part name="D7" library="zetex" library_urn="urn:adsk.eagle:library:418" deviceset="D" device="SOD323" package3d_urn="urn:adsk.eagle:package:30992/1"/>
-<part name="D8" library="zetex" library_urn="urn:adsk.eagle:library:418" deviceset="D" device="SOD323" package3d_urn="urn:adsk.eagle:package:30992/1"/>
+<part name="D1" library="zetex" library_urn="urn:adsk.eagle:library:418" deviceset="D" device="SOD323" package3d_urn="urn:adsk.eagle:package:30992/1"/>
+<part name="D2" library="zetex" library_urn="urn:adsk.eagle:library:418" deviceset="D" device="SOD323" package3d_urn="urn:adsk.eagle:package:30992/1"/>
 <part name="R3" library="resistor" deviceset="R-US_" device="R0402" value="220R"/>
 <part name="CN3" library="resistor" deviceset="CNET" device="" value="100nF"/>
@@
 <part name="IC2" library="CPSS_IC" deviceset="W25N01GVZEIG/IT" device=""/>
 <part name="XU1" library="CPSS_CONNECTOR" deviceset="MICROUSB_5POS_SMT" device=""/>
-<part name="J2" library="SparkFun-Connectors" library_urn="urn:adsk.eagle:library:513" deviceset="CONN_02" device="" package3d_urn="urn:adsk.eagle:package:38039/1"/>
+<part name="JP3" library="SparkFun-Connectors" library_urn="urn:adsk.eagle:library:513" deviceset="CONN_02" device="" package3d_urn="urn:adsk.eagle:package:38039/1"/>
 <part name="R4" library="resistor" deviceset="R-US_" device="R0402" value="220R"/>
 <part name="GND6" library="supply1" library_urn="urn:adsk.eagle:library:371" deviceset="GND" device=""/>
 <part name="C7" library="resistor" deviceset="C-EU" device="C0603" value="100n"/>
 <part name="RN1" library="resistor-net" library_urn="urn:adsk.eagle:library:343" deviceset="CTS742C083" device="" package3d_urn="urn:adsk.eagle:package:24985/1" value="65R"/>
-<part name="U$6" library="CPSS_CONNECTOR" deviceset="SOLBRDG" device=""/>
-<part name="U$7" library="CPSS_CONNECTOR" deviceset="SOLBRDG" device=""/>
+<part name="SJ3" library="CPSS_CONNECTOR" deviceset="SOLBRDG" device=""/>
+<part name="SJ2" library="CPSS_CONNECTOR" deviceset="SOLBRDG" device=""/>
 <part name="Q1" library="CPSS_IC" deviceset="MBT3904DW2T1" device=""/>
 <part name="Q2" library="CPSS_IC" deviceset="MBT3904DW2T1" device=""/>
@@
 <attribute name="NAME" x="140.97" y="262.89" size="3.81" layer="95"/>
 </instance>
-<instance part="U$2" gate="G$1" x="53.34" y="128.27"/>
+<instance part="SD1" gate="G$1" x="53.34" y="128.27"/>
 <instance part="XP1" gate="G$1" x="20.32" y="43.18"/>
 <instance part="R1" gate="G$1" x="125.73" y="74.93"/>
@@
 <instance part="C1" gate="G$1" x="133.35" y="199.39"/>
 <instance part="R5" gate="G$1" x="125.73" y="196.85" rot="R90"/>
-<instance part="D7" gate="G$1" x="292.1" y="255.27"/>
-<instance part="D8" gate="G$1" x="292.1" y="245.11"/>
+<instance part="D1" gate="G$1" x="292.1" y="255.27"/>
+<instance part="D2" gate="G$1" x="292.1" y="245.11"/>
 <instance part="R3" gate="G$1" x="287.02" y="99.06"/>
 <instance part="CN3" gate="G$1" x="133.35" y="38.1"/>
@@
 <instance part="IC2" gate="G$1" x="347.98" y="101.6"/>
 <instance part="XU1" gate="G$1" x="20.32" y="76.2" rot="R90"/>
-<instance part="J2" gate="G$1" x="330.2" y="83.82" rot="R180"/>
+<instance part="JP3" gate="G$1" x="330.2" y="83.82" rot="R180"/>
 <instance part="R4" gate="G$1" x="347.98" y="111.76"/>
 <instance part="GND6" gate="1" x="342.9" y="83.82"/>
 <instance part="C7" gate="G$1" x="360.68" y="88.9" rot="R90"/>
 <instance part="RN1" gate="G$1" x="292.1" y="210.82"/>
-<instance part="U$6" gate="G$1" x="262.89" y="158.75"/>
-<instance part="U$7" gate="G$1" x="270.51" y="168.91"/>
+<instance part="SJ3" gate="G$1" x="262.89" y="158.75"/>
+<instance part="SJ2" gate="G$1" x="270.51" y="168.91"/>
 <instance part="Q1" gate="G$1" x="316.23" y="195.58" smashed="yes" rot="R90">
 <attribute name="NAME" x="312.42" y="199.39" size="1.778" layer="95"/>
@@
 </segment>
 <segment>
-<pinref part="U$2" gate="G$1" pin="3-CMO"/>
+<pinref part="SD1" gate="G$1" pin="3-CMO"/>
 <wire x1="40.64" y1="135.89" x2="33.02" y2="135.89" width="0.1524" layer="91"/>
 <label x="33.02" y="135.89" size="1.778" layer="95"/>
@@
 </segment>
 <segment>
-<pinref part="U$2" gate="G$1" pin="4-VDD"/>
+<pinref part="SD1" gate="G$1" pin="4-VDD"/>
 <wire x1="40.64" y1="130.81" x2="33.02" y2="130.81" width="0.1524" layer="91"/>
 <label x="33.02" y="130.81" size="1.778" layer="95"/>
@@
 <wire x1="270.51" y1="163.83" x2="270.51" y2="158.75" width="0.1524" layer="91"/>
 <junction x="270.51" y="158.75"/>
-<pinref part="U$6" gate="G$1" pin="P$2"/>
+<pinref part="SJ3" gate="G$1" pin="P$2"/>
 </segment>
 <segment>
@@
 </segment>
 <segment>
-<pinref part="U$2" gate="G$1" pin="GND1"/>
+<pinref part="SD1" gate="G$1" pin="GND1"/>
 <wire x1="73.66" y1="146.05" x2="78.74" y2="146.05" width="0.1524" layer="91"/>
 <wire x1="78.74" y1="146.05" x2="78.74" y2="135.89" width="0.1524" layer="91"/>
-<pinref part="U$2" gate="G$1" pin="GND2"/>
+<pinref part="SD1" gate="G$1" pin="GND2"/>
 <wire x1="78.74" y1="135.89" x2="73.66" y2="135.89" width="0.1524" layer="91"/>
 <wire x1="78.74" y1="135.89" x2="78.74" y2="125.73" width="0.1524" layer="91"/>
 <junction x="78.74" y="135.89"/>
-<pinref part="U$2" gate="G$1" pin="GND3"/>
+<pinref part="SD1" gate="G$1" pin="GND3"/>
 <wire x1="78.74" y1="125.73" x2="73.66" y2="125.73" width="0.1524" layer="91"/>
 <wire x1="78.74" y1="125.73" x2="78.74" y2="123.19" width="0.1524" layer="91"/>
@@
 </segment>
 <segment>
-<pinref part="U$2" gate="G$1" pin="6-VSS"/>
+<pinref part="SD1" gate="G$1" pin="6-VSS"/>
 <wire x1="40.64" y1="120.65" x2="33.02" y2="120.65" width="0.1524" layer="91"/>
 <label x="33.02" y="120.65" size="1.778" layer="95"/>
@@
 <pinref part="GND2" gate="1" pin="GND"/>
 <wire x1="275.59" y1="168.91" x2="283.21" y2="168.91" width="0.1524" layer="91"/>
-<pinref part="U$7" gate="G$1" pin="P$2"/>
+<pinref part="SJ2" gate="G$1" pin="P$2"/>
 </segment>
 <segment>
@@
 </segment>
 <segment>
-<pinref part="U$2" gate="G$1" pin="5-CLK"/>
+<pinref part="SD1" gate="G$1" pin="5-CLK"/>
 <wire x1="40.64" y1="125.73" x2="33.02" y2="125.73" width="0.1524" layer="91"/>
 <label x="33.02" y="125.73" size="1.778" layer="95"/>
@@
 </segment>
 <segment>
-<pinref part="U$2" gate="G$1" pin="7-DAT0"/>
+<pinref part="SD1" gate="G$1" pin="7-DAT0"/>
 <wire x1="40.64" y1="115.57" x2="33.02" y2="115.57" width="0.1524" layer="91"/>
 <label x="33.02" y="115.57" size="1.778" layer="95"/>
@@
 <segment>
 <label x="312.42" y="104.14" size="1.778" layer="95"/>
-<pinref part="J2" gate="G$1" pin="1"/>
+<pinref part="JP3" gate="G$1" pin="1"/>
 <wire x1="320.04" y1="104.14" x2="312.42" y2="104.14" width="0.1524" layer="91"/>
 <wire x1="320.04" y1="104.14" x2="320.04" y2="83.82" width="0.1524" layer="91"/>
@@
 <segment>
 <label x="312.42" y="99.06" size="1.778" layer="95"/>
-<pinref part="J2" gate="G$1" pin="2"/>
+<pinref part="JP3" gate="G$1" pin="2"/>
 <wire x1="317.5" y1="99.06" x2="312.42" y2="99.06" width="0.1524" layer="91"/>
 <wire x1="317.5" y1="99.06" x2="317.5" y2="81.28" width="0.1524" layer="91"/>
@@
 <net name="5V" class="4">
 <segment>
-<pinref part="D8" gate="G$1" pin="A"/>
+<pinref part="D2" gate="G$1" pin="A"/>
 <wire x1="289.56" y1="245.11" x2="284.48" y2="245.11" width="0.1524" layer="91"/>
 <label x="284.48" y="245.11" size="1.778" layer="95"/>
@@
 <pinref part="ERASE" gate="G$1" pin="P$1"/>
 <wire x1="248.92" y1="158.75" x2="257.81" y2="158.75" width="0.1524" layer="91"/>
-<pinref part="U$6" gate="G$1" pin="P$1"/>
+<pinref part="SJ3" gate="G$1" pin="P$1"/>
 </segment>
 </net>
@@
 <pinref part="RESET" gate="G$1" pin="P$1"/>
 <wire x1="260.35" y1="168.91" x2="265.43" y2="168.91" width="0.1524" layer="91"/>
-<pinref part="U$7" gate="G$1" pin="P$1"/>
+<pinref part="SJ2" gate="G$1" pin="P$1"/>
 </segment>
 </net>
@@
 <junction x="297.18" y="250.19"/>
 <wire x1="297.18" y1="245.11" x2="294.64" y2="245.11" width="0.1524" layer="91"/>
-<pinref part="D7" gate="G$1" pin="C"/>
-<pinref part="D8" gate="G$1" pin="C"/>
+<pinref part="D1" gate="G$1" pin="C"/>
+<pinref part="D2" gate="G$1" pin="C"/>
 </segment>
 </net>
@@
 </segment>
 <segment>
-<pinref part="D7" gate="G$1" pin="A"/>
+<pinref part="D1" gate="G$1" pin="A"/>
 <wire x1="289.56" y1="255.27" x2="284.48" y2="255.27" width="0.1524" layer="91"/>
 <label x="284.48" y="255.27" size="1.778" layer="95"/>
@@
 </segment>
 <segment>
-<pinref part="U$2" gate="G$1" pin="2-CD/DAT3"/>
+<pinref part="SD1" gate="G$1" pin="2-CD/DAT3"/>
 <wire x1="40.64" y1="140.97" x2="33.02" y2="140.97" width="0.1524" layer="91"/>
 <label x="33.02" y="140.97" size="1.778" layer="95"/>
