File: CubeStack/Sensor Board/SB2.brd (EAGLE design)
At the start: 63.5 x 76.2 mm, 21 parts, among them U1 LSM6DSL, U2 LSM6DSL, U3 H3LIS331DL, U4 LIS2MDL, U5 MS56XX-0XBA0X

Commit message: Update SB2.brd
Routing:
- net GND: vias 83 -> 111
Other:
- board text added: "1 11 21 31"
Changed lines of the file:
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@@
 <dimension x1="31.75" y1="46.99" x2="46.736" y2="46.99" x3="39.243" y3="48.768" textsize="0.8128" layer="21" precision="0"/>
 <dimension x1="29.21" y1="44.45" x2="29.21" y2="29.464" x3="27.050996875" y3="36.957" textsize="0.8128" layer="21" precision="0"/>
+<text x="18.288" y="55.372" size="0.8636" layer="21" align="bottom-right">1
+11
+21
+31</text>
 </plain>
 <attributes>
@@
 </element>
 <element name="U2" library="CPSS_SENSOR" package="LGA-14" value="LSM6DSL" x="31.75" y="29.591" smashed="yes">
-<attribute name="NAME" x="36.37" y="26.241" size="0.8128" layer="25"/>
+<attribute name="NAME" x="27.988" y="28.273" size="0.8128" layer="25"/>
 </element>
 <element name="U5" library="CPSS_SENSOR" package="MS56XX" value="MS56XX-0XBA0X" x="46.736" y="26.162" smashed="yes" rot="R270">
-<attribute name="NAME" x="51.736" y="28.162" size="0.8128" layer="25" rot="R270"/>
+<attribute name="NAME" x="42.45" y="25.828" size="0.8128" layer="25"/>
 </element>
 <element name="U3" library="CPSS_SENSOR" package="TFLGA-16L" value="H3LIS331DL" x="46.736" y="44.45" smashed="yes" rot="R180">
@@
 </element>
 <element name="C3" library="rcl" library_urn="urn:adsk.eagle:library:334" package="C0805" package3d_urn="urn:adsk.eagle:package:23617/2" value="100n" x="31.75" y="26.416" smashed="yes">
-<attribute name="NAME" x="30.48" y="27.686" size="0.8128" layer="25"/>
+<attribute name="NAME" x="28.702" y="24.384" size="0.8128" layer="25"/>
 <attribute name="SPICEPREFIX" value="C" x="31.75" y="26.416" size="0.8128" layer="27" display="off"/>
 </element>
 <element name="C4" library="rcl" library_urn="urn:adsk.eagle:library:334" package="C0805" package3d_urn="urn:adsk.eagle:package:23617/2" value="100n" x="35.56" y="27.94" smashed="yes" rot="R270">
-<attribute name="NAME" x="36.83" y="29.21" size="0.8128" layer="25" rot="R270"/>
+<attribute name="NAME" x="36.83" y="27.686" size="0.8128" layer="25"/>
 <attribute name="SPICEPREFIX" value="C" x="35.56" y="27.94" size="0.8128" layer="27" rot="R270" display="off"/>
 </element>
@@
 </element>
 <element name="C7" library="rcl" library_urn="urn:adsk.eagle:library:334" package="C0805" package3d_urn="urn:adsk.eagle:package:23617/2" value="100n" x="46.482" y="29.718" smashed="yes" rot="R180">
-<attribute name="NAME" x="47.752" y="28.448" size="0.8128" layer="25" rot="R180"/>
+<attribute name="NAME" x="50.038" y="30.226" size="0.8128" layer="25" rot="R180"/>
 <attribute name="SPICEPREFIX" value="C" x="46.482" y="29.718" size="0.8128" layer="27" rot="R180" display="off"/>
 </element>
@@
 <via x="62.738" y="68.326" extent="1-16" drill="0.35"/>
 <via x="62.738" y="71.882" extent="1-16" drill="0.35"/>
+<via x="54.864" y="52.324" extent="1-16" drill="0.35"/>
+<via x="54.864" y="48.006" extent="1-16" drill="0.35"/>
+<via x="54.864" y="42.164" extent="1-16" drill="0.35"/>
+<via x="54.864" y="36.068" extent="1-16" drill="0.35"/>
+<via x="54.864" y="29.972" extent="1-16" drill="0.35"/>
+<via x="54.864" y="24.13" extent="1-16" drill="0.35"/>
+<via x="49.784" y="19.558" extent="1-16" drill="0.35"/>
+<via x="54.864" y="19.558" extent="1-16" drill="0.35"/>
+<via x="43.688" y="19.558" extent="1-16" drill="0.35"/>
+<via x="37.846" y="19.558" extent="1-16" drill="0.35"/>
+<via x="31.75" y="19.558" extent="1-16" drill="0.35"/>
+<via x="25.654" y="19.558" extent="1-16" drill="0.35"/>
+<via x="19.558" y="19.558" extent="1-16" drill="0.35"/>
+<via x="13.716" y="19.558" extent="1-16" drill="0.35"/>
+<via x="8.382" y="19.558" extent="1-16" drill="0.35"/>
+<via x="8.382" y="23.876" extent="1-16" drill="0.35"/>
+<via x="8.382" y="29.972" extent="1-16" drill="0.35"/>
+<via x="8.382" y="36.068" extent="1-16" drill="0.35"/>
+<via x="8.382" y="41.91" extent="1-16" drill="0.35"/>
+<via x="8.382" y="48.006" extent="1-16" drill="0.35"/>
+<via x="13.716" y="52.324" extent="1-16" drill="0.35"/>
+<via x="8.382" y="52.324" extent="1-16" drill="0.35"/>
+<via x="19.304" y="52.324" extent="1-16" drill="0.35"/>
+<via x="25.146" y="52.324" extent="1-16" drill="0.35"/>
+<via x="42.926" y="52.324" extent="1-16" drill="0.35"/>
+<via x="49.53" y="52.324" extent="1-16" drill="0.35"/>
+<via x="30.988" y="52.324" extent="1-16" drill="0.35"/>
+<via x="32.512" y="52.324" extent="1-16" drill="0.35"/>
 </signal>
 <signal name="5V">
@@
 </drawing>
 <compatibility>
+<note version="6.3" minversion="6.2.2" severity="warning">
+Since Version 6.2.2 text objects can contain more than one line,
+which will not be processed correctly with this version.
+</note>
 <note version="8.2" severity="warning">
 Since Version 8.2, EAGLE supports online libraries. The ids
